File: KiCAD/XIAOC6_Occupancy_Battery.kicad_sch (KiCad schematic)
At the start: 6 parts, among them U1 ZC362800_, U2 XIAO-ESP32-S3-SMD, U3 SHTC3

Commit message: update
Parts:
- added J1: Conn_01x02_Socket, Connector_JST:JST_PH_S2B-PH-K_1x02_P2.00mm_Horizontal, symbol Connector:Conn_01x02_Socket
- U3: footprint Sensor:ASAIR_AM2302_P2.54mm_Vertical -> Sensor:ASAIR_AM2302_P2.54mm_Lead2.75mm_TabDown
Connections:
- net +BATT: now also J1.2 (Pin_2)
- net -BATT: now also J1.1 (Pin_1)
